File: PCBs/drawing_machine_controller/drawing_machine_controller.kicad_sch (KiCad schematic)
At the start: 28 parts, among them J1 USB_C_Receptacle_USB2.0, J2 USB_C_Receptacle_USB2.0, J3 USB_C_Receptacle_USB2.0, J4 USB_C_Receptacle_USB2.0, Q1 AO3400A, U1 ESP32-DEVKIT-V1, U2 IP2721, U3 TMC2130_V3_BIGTREETECH, U4 TMC2130_V3_BIGTREETECH, U5 TMC2130_V3_BIGTREETECH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

Commit message: pcb tweak, fluidnc start
Parts:
- C1, C4, C5: footprint Capacitor_SMD:CP_Elec_6.3x7.7 -> Capacitor_SMD:CP_Elec_8x6.7
